Commit message: add gripper tcp_xyz tcp_rpy as params

File: robotiq/robotiq_description/urdf/robotiq_85_gripper.urdf.xacro (robot description, xacro)
@@ -2,5 +2,5 @@
 <robot name="robotiq_85_gripper" xmlns:xacro="http://www.ros.org/wiki/xacro">
   <xacro:include filename="$(find robotiq_description)/urdf/robotiq_85_gripper.transmission.xacro" />
-  <xacro:macro name="robotiq_85_gripper" params="prefix parent *origin">
+  <xacro:macro name="robotiq_85_gripper" params="prefix parent *origin tcp_xyz:='0.15 0 0' tcp_rpy:='0 0 0'">
     <joint name="${prefix}robotiq_85_base_joint" type="fixed">
       <parent link="${parent}"/>
@@ -30,5 +30,5 @@
     <link name="${prefix}ur5_gripper_tcp" />
     <joint name="${prefix}ur5_gripper_tcp_joint" type="fixed">
-      <origin xyz="0.15 0 0.0" rpy="0 0 0" />
+      <origin xyz="${tcp_xyz}" rpy="${tcp_rpy}" />
       <parent link="${prefix}robotiq_85_base_link"/>
       <child link="${prefix}ur5_gripper_tcp"/>
